Commit message: Enhance gazebo.xacro with detailed sensor configurations for camera, LIDAR, and IMU; improve structure with section headers for clarity

File: src/my_robot_description/urdf/urdf/gazebo.xacro (robot description, xacro)
@@ -1,5 +1,7 @@
 <?xml version="1.0"?>
 <robot xmlns:xacro="http://www.ros.org/wiki/xacro">
-    <!-- Gazebo ROS2 Control -->
+    <!-- ===================================================== -->
+    <!-- GAZEBO ROS2 CONTROL -->
+    <!-- ===================================================== -->
     <gazebo>
         <plugin
@@ -8,16 +10,16 @@
         </plugin>
     </gazebo>
-    <!-- WHEEL 1 -->
+    <!-- ===================================================== -->
+    <!-- WHEEL PHYSICS -->
+    <!-- ===================================================== -->
+    <!-- RIGHT WHEEL 1 -->
     <gazebo reference="right_wheel_1_link">
-        <!-- Fricción mecanum -->
         <mu1>0.05</mu1>
         <mu2>1.0</mu2>
-        <!-- Física -->
         <kp>1000000.0</kp>
         <kd>100.0</kd>
-        <!-- Material -->
         <material>Gazebo/Black</material>
     </gazebo>
-    <!-- WHEEL 2 -->
+    <!-- RIGHT WHEEL 2 -->
     <gazebo reference="right_wheel_2_link">
         <mu1>0.05</mu1>
@@ -27,5 +29,5 @@
         <material>Gazebo/Black</material>
     </gazebo>
-    <!-- WHEEL 3 -->
+    <!-- LEFT WHEEL 1 -->
     <gazebo reference="left_wheel_1_link">
         <mu1>0.05</mu1>
@@ -35,5 +37,5 @@
         <material>Gazebo/Black</material>
     </gazebo>
-    <!-- WHEEL 4 -->
+    <!-- LEFT WHEEL 2 -->
     <gazebo reference="left_wheel_2_link">
         <mu1>0.05</mu1>
@@ -43,3 +45,112 @@
         <material>Gazebo/Black</material>
     </gazebo>
+    <!-- ===================================================== -->
+    <!-- CAMERA -->
+    <!-- ===================================================== -->
+    <gazebo reference="elp_1080p_link">
+        <sensor name="camera_sensor" type="camera">
+            <always_on>true</always_on>
+            <update_rate>30</update_rate>
+            <visualize>true</visualize>
+            <camera>
+                <horizontal_fov>1.5708</horizontal_fov>
+                <image>
+                    <width>1920</width>
+                    <height>1080</height>
+                    <format>R8G8B8</format>
+                </image>
+                <clip>
+                    <near>0.05</near>
+                    <far>100</far>
+                </clip>
+            </camera>
+            <plugin
+                name="camera_controller"
+                filename="libgazebo_ros_camera.so">
+                <ros>
+                    <namespace>/camera</namespace>
+                    <remapping>image_raw:=image_raw</remapping>
+                    <remapping>camera_info:=camera_info</remapping>
+                </ros>
+                <frame_name>elp_1080p_link</frame_name>
+            </plugin>
+        </sensor>
+    </gazebo>
+    <!-- ===================================================== -->
+    <!-- LIDAR -->
+    <!-- ===================================================== -->
+    <gazebo reference="sensor_lidar_link">
+        <sensor name="lidar_sensor" type="ray">
+            <always_on>true</always_on>
+            <update_rate>15</update_rate>
+            <visualize>true</visualize>
+            <ray>
+                <scan>
+                    <horizontal>
+                        <samples>720</samples>
+                        <resolution>1</resolution>
+                        <min_angle>-3.14159</min_angle>
+                        <max_angle>3.14159</max_angle>
+                    </horizontal>
+                </scan>
+                <range>
+                    <min>0.10</min>
+                    <max>12.0</max>
+                    <resolution>0.01</resolution>
+                </range>
+            </ray>
+            <plugin
+                name="lidar_plugin"
+                filename="libgazebo_ros_ray_sensor.so">
+                <ros>
+                    <namespace>/lidar</namespace>
+                    <remapping>~/out:=scan</remapping>
+                </ros>
+                <output_type>sensor_msgs/LaserScan</output_type>
+                <frame_name>sensor_lidar_link</frame_name>
+            </plugin>
+        </sensor>
+    </gazebo>
+    <!-- ===================================================== -->
+    <!-- IMU -->
+    <!-- ===================================================== -->
+    <gazebo reference="base_link">
+        <sensor name="imu_sensor" type="imu">
+            <always_on>true</always_on>
+            <update_rate>100</update_rate>
+            <plugin
+                name="imu_plugin"
+                filename="libgazebo_ros_imu_sensor.so">
+                <ros>
+                    <namespace>/imu</namespace>
+                    <remapping>~/out:=data</remapping>
+                </ros>
+                <frame_name>base_link</frame_name>
+            </plugin>
+        </sensor>
+    </gazebo>
+    <!-- ===================================================== -->
+    <!-- SCREEN (VISUAL ONLY) -->
+    <!-- ===================================================== -->
+    <gazebo reference="pantalla_link">
+        <material>Gazebo/Blue</material>
+    </gazebo>
+    <!-- ===================================================== -->
+    <!-- SPEAKERS (VISUAL ONLY) -->
+    <!-- ===================================================== -->
+    <gazebo reference="altavoz_3_link">
+        <material>Gazebo/DarkGrey</material>
+    </gazebo>
+    <gazebo reference="altavoz_3_2_link">
+        <material>Gazebo/DarkGrey</material>
+    </gazebo>
+    <!-- ===================================================== -->
+    <!-- MICROPHONES (VISUAL ONLY) -->
+    <!-- ===================================================== -->
+    <gazebo reference="matriz_de_microfono_resaker_12v_link">
+        <material>Gazebo/Grey</material>
+    </gazebo>
+    <gazebo reference="matriz_de_microfono_resaker_12v_1_link">
+        <material>Gazebo/Grey</material>
+    </gazebo>
 </robot>
