Commit message: Add color properties for screen, altavoz, electronics, and lidar in parameter.xacro

File: src/my_robot_description/urdf/urdf/parameter.xacro (robot description, xacro)
@@ -7,3 +7,11 @@
     <xacro:property name="name_color_wheel" value="yellow"/>
     <xacro:property name="rgba_wheel" value="1 1 0 1"/>
+    <xacro:property name="name_color_screen" value="black"/>
+    <xacro:property name="rgba_screen" value="0 0 0 1"/>
+    <xacro:property name="name_color_altavoz" value="gray"/>
+    <xacro:property name="rgba_altavoz" value="0.5 0.5 0.5 1"/>
+    <xacro:property name="name_color_electronics" value="black"/>
+    <xacro:property name="rgba_electronics" value="0 0 0 1"/>
+    <xacro:property name="name_color_lidar" value="Pinkish_red"/>
+    <xacro:property name="rgba_lidar" value="1 0.4 0.4 1"/>
 </robot>
