Commit message: Refactor joint names and comments in ros2_control.xacro for clarity

File: src/my_robot_description/urdf/urdf/ros2_control.xacro (robot description, xacro)
@@ -5,14 +5,5 @@
             <plugin>gazebo_ros2_control/GazeboSystem</plugin>
         </hardware>
-        <!-- Wheel 1 -->
-        <joint name="base_link_to_right_wheel_1">
-            <command_interface name="velocity">
-                <param name="min">-20</param>
-                <param name="max">20</param>
-            </command_interface>
-            <state_interface name="position"/>
-            <state_interface name="velocity"/>
-        </joint>
-        <!-- Wheel 2 -->
+        <!-- RIGHT WHEEL FRONT -->
         <joint name="base_link_to_right_wheel_2">
             <command_interface name="velocity">
@@ -23,6 +14,6 @@
             <state_interface name="velocity"/>
         </joint>
-        <!-- Wheel 3 -->
-        <joint name="base_link_to_left_wheel_3">
+        <!-- RIGHT WHEEL REAR -->
+        <joint name="base_link_to_right_wheel_3">
             <command_interface name="velocity">
                 <param name="min">-20</param>
@@ -32,5 +23,14 @@
             <state_interface name="velocity"/>
         </joint>
-        <!-- Wheel 4 -->
+        <!-- LEFT WHEEL FRONT -->
+        <joint name="base_link_to_left_wheel_1">
+            <command_interface name="velocity">
+                <param name="min">-20</param>
+                <param name="max">20</param>
+            </command_interface>
+            <state_interface name="position"/>
+            <state_interface name="velocity"/>
+        </joint>
+        <!-- LEFT WHEEL REAR -->
         <joint name="base_link_to_left_wheel_4">
             <command_interface name="velocity">
