Commit message: Update scale parameters for mesh and collision geometry in macro.xacro

File: src/my_robot_description/urdf/urdf/macro.xacro (robot description, xacro)
@@ -10,5 +10,5 @@
                 <geometry>
                     <mesh filename="../stl/${name_folder}/${name}.stl"
-                scale="1 1 1"/>
+                scale="0.001 0.001 0.001"/>
                 </geometry>
                 <material name="${name_color}">
@@ -20,5 +20,5 @@
                 <geometry>
                     <mesh filename="../stl/${name_folder}/${name}.stl"
-                scale="1 1 1"/>
+                        scale="0.001 0.001 0.001"/>
                 </geometry>
             </collision>
@@ -35,5 +35,5 @@
     <xacro:macro
         name="create_link_wheel"
-        params="name name_link name_folder name_color rgba"
+        params="name name_link name_folder name_color rgba xyz_collition"
         >
             <link name="${name_link}">
@@ -43,5 +43,5 @@
                     <geometry>
                         <mesh filename="../stl/${name_folder}/${name}.stl"
-                            scale="1 1 1"/>
+                            scale="0.001 0.001 0.001"/>
                     </geometry>
                     <material name="${name_color}">
@@ -51,7 +51,7 @@
                 <!-- COLLISION -->
                 <collision>
-                    <origin xyz="0 0 0" rpy="0 0 0"/>
+                    <origin xyz="${xyz_collition}" rpy="1.5708 0 0"/>
                     <geometry>
-                        <cylinder length="0.5" radius="0.1" scale="1 1 1"/>
+                        <cylinder length="0.045674" radius="0.028885"/>
                     </geometry>
                 </collision>
@@ -68,6 +68,6 @@
                         izz="0.001"/>
                 </inertial>
-    </link>
-</xacro:macro>
+        </link>
+    </xacro:macro>
     <xacro:macro
         name="create_joint_fixed"

Commit message: Fix mesh file paths in macro.xacro for correct URDF representation

File: src/my_robot_description/urdf/urdf/macro.xacro (robot description, xacro)
@@ -9,5 +9,5 @@
                 <origin xyz="${xyz}" rpy="${rpy}"/>
                 <geometry>
-                    <mesh filename="../stl/${name_folder}/${name}.stl"
+                    <mesh filename="package://my_robot_description/urdf/stl/${name_folder}/${name}.stl"
                 scale="0.001 0.001 0.001"/>
                 </geometry>
@@ -19,5 +19,5 @@
                 <origin xyz="${xyz}" rpy="${rpy}"/>
                 <geometry>
-                    <mesh filename="../stl/${name_folder}/${name}.stl"
+                    <mesh filename="package://my_robot_description/urdf/stl/${name_folder}/${name}.stl"
                         scale="0.001 0.001 0.001"/>
                 </geometry>
@@ -42,5 +42,5 @@
                     <origin xyz="0 0 0" rpy="0 0 0"/>
                     <geometry>
-                        <mesh filename="../stl/${name_folder}/${name}.stl"
+                        <mesh filename="package://my_robot_description/urdf/stl/${name_folder}/${name}.stl"
                             scale="0.001 0.001 0.001"/>
                     </geometry>

Commit message: Fix parameter list and origin rpy in create_link_wheel and create_joint_continuous macros

File: src/my_robot_description/urdf/urdf/macro.xacro (robot description, xacro)
@@ -35,5 +35,5 @@
     <xacro:macro
         name="create_link_wheel"
-        params="name name_link name_folder name_color rgba xyz_collition"
+        params="name name_link name_folder name_color rgba xyz_collition rpy"
         >
             <link name="${name_link}">
@@ -51,5 +51,5 @@
                 <!-- COLLISION -->
                 <collision>
-                    <origin xyz="${xyz_collition}" rpy="1.5708 0 0"/>
+                    <origin xyz="${xyz_collition}" rpy="${rpy}"/>
                     <geometry>
                         <cylinder length="0.045674" radius="0.028885"/>
@@ -82,5 +82,5 @@
     <xacro:macro
         name="create_joint_continuous"
-        params="name parent child xyz rpy axis limit_lower limit_upper">
+        params="name parent child xyz rpy axis">
         <joint name="${name}" type="continuous">
             <parent link="${parent}"/>

Commit message: Refactor macro.xacro to improve link and joint definitions; streamline mesh file paths and remove commented-out inertial properties

File: src/my_robot_description/urdf/urdf/macro.xacro (robot description, xacro)
@@ -1,14 +1,10 @@
 <?xml version="1.0" ?>
 <robot name="my_robot" xmlns:xacro="http://www.ros.org/wiki/xacro">
-    <xacro:macro
-    name="create_link"
-    params= "name name_link name_folder name_color rgba xyz rpy"
-    >
+    <xacro:macro name="create_link" params="name name_link name_folder name_color rgba xyz rpy stl_path">
         <link name="${name_link}">
             <visual>
                 <origin xyz="${xyz}" rpy="${rpy}"/>
                 <geometry>
-                    <mesh filename="package://my_robot_description/urdf/stl/${name_folder}/${name}.stl"
-                scale="0.001 0.001 0.001"/>
+                    <mesh filename="${stl_path}/${name_folder}/${name}.stl" scale="0.001 0.001 0.001"/>
                 </geometry>
                 <material name="${name_color}">
@@ -19,59 +15,39 @@
                 <origin xyz="${xyz}" rpy="${rpy}"/>
                 <geometry>
-                    <mesh filename="package://my_robot_description/urdf/stl/${name_folder}/${name}.stl"
-                        scale="0.001 0.001 0.001"/>
+                    <mesh filename="${stl_path}/${name_folder}/${name}.stl" scale="0.001 0.001 0.001"/>
                 </geometry>
             </collision>
-            <!-- <inertial>
-                <mass value="${inertial_mass}"/>
+            <inertial>
+                <mass value="0.05"/>
                 <origin xyz="${xyz}" rpy="${rpy}"/>
-                <inertia
-                    ixx="${inertial_ixx}" ixy="0.0" ixz="0.0"
-                    iyy="${inertial_iyy}" iyz="0.0"
-                    izz="${inertial_izz}"/>
-            </inertial> -->
+                <inertia ixx="0.001" ixy="0.0" ixz="0.0" iyy="0.001" iyz="0.0" izz="0.001"/>
+            </inertial>
         </link>
     </xacro:macro>
-    <xacro:macro
-        name="create_link_wheel"
-        params="name name_link name_folder name_color rgba xyz_collition rpy"
-        >
-            <link name="${name_link}">
-                <!-- VISUAL -->
-                <visual>
-                    <origin xyz="0 0 0" rpy="0 0 0"/>
-                    <geometry>
-                        <mesh filename="package://my_robot_description/urdf/stl/${name_folder}/${name}.stl"
-                            scale="0.001 0.001 0.001"/>
-                    </geometry>
-                    <material name="${name_color}">
-                        <color rgba="${rgba}"/>
-                    </material>
-                </visual>
-                <!-- COLLISION -->
-                <collision>
-                    <origin xyz="${xyz_collition}" rpy="${rpy}"/>
-                    <geometry>
-                        <cylinder length="0.045674" radius="0.028885"/>
-                    </geometry>
-                </collision>
-                <!-- INERTIA -->
-                <inertial>
-                    <mass value="0.5"/>
-                    <origin xyz="0 0 0" rpy="0 0 0"/>
-                    <inertia
-                        ixx="0.001"
-                        ixy="0.0"
-                        ixz="0.0"
-                        iyy="0.001"
-                        iyz="0.0"
-                        izz="0.001"/>
-                </inertial>
+    <xacro:macro name="create_link_wheel" params="name name_link name_folder name_color rgba xyz_collition rpy stl_path">
+        <link name="${name_link}">
+            <visual>
+                <origin xyz="0 0 0" rpy="0 0 0"/>
+                <geometry>
+                    <mesh filename="${stl_path}/${name_folder}/${name}.stl" scale="0.001 0.001 0.001"/>
+                </geometry>
+                <material name="${name_color}">
+                    <color rgba="${rgba}"/>
+                </material>
+            </visual>
+            <collision>
+                <origin xyz="${xyz_collition}" rpy="${rpy}"/>
+                <geometry>
+                    <cylinder length="0.045674" radius="0.028885"/>
+                </geometry>
+            </collision>
+            <inertial>
+                <mass value="0.5"/>
+                <origin xyz="0 0 0" rpy="0 0 0"/>
+                <inertia ixx="0.001" ixy="0.0" ixz="0.0" iyy="0.001" iyz="0.0" izz="0.001"/>
+            </inertial>
         </link>
     </xacro:macro>
-    <xacro:macro
-        name="create_joint_fixed"
-        params="name parent child xyz rpy"
-    >
+    <xacro:macro name="create_joint_fixed" params="name parent child xyz rpy">
         <joint name="${name}" type="fixed">
             <parent link="${parent}"/>
@@ -80,7 +56,5 @@
         </joint>
     </xacro:macro>
-    <xacro:macro
-        name="create_joint_continuous"
-        params="name parent child xyz rpy axis">
+    <xacro:macro name="create_joint_continuous" params="name parent child xyz rpy axis">
         <joint name="${name}" type="continuous">
             <parent link="${parent}"/>

Commit message: Refactor macro.xacro and parameter.xacro to enhance mass property definitions; update robot.xacro to utilize new mass parameters for improved link creation

File: src/my_robot_description/urdf/urdf/macro.xacro (robot description, xacro)
@@ -1,5 +1,5 @@
 <?xml version="1.0" ?>
 <robot name="my_robot" xmlns:xacro="http://www.ros.org/wiki/xacro">
-    <xacro:macro name="create_link" params="name name_link name_folder name_color rgba xyz rpy stl_path">
+    <xacro:macro name="create_link" params="name name_link name_folder name_color rgba xyz rpy stl_path mass">
         <link name="${name_link}">
             <visual>
@@ -19,5 +19,5 @@
             </collision>
             <inertial>
-                <mass value="0.05"/>
+                <mass value="${mass}"/>
                 <origin xyz="${xyz}" rpy="${rpy}"/>
                 <inertia ixx="0.001" ixy="0.0" ixz="0.0" iyy="0.001" iyz="0.0" izz="0.001"/>
@@ -43,5 +43,5 @@
             </collision>
             <inertial>
-                <mass value="0.5"/>
+                <mass value="0.045267"/>
                 <origin xyz="0 0 0" rpy="0 0 0"/>
                 <inertia ixx="0.001" ixy="0.0" ixz="0.0" iyy="0.001" iyz="0.0" izz="0.001"/>

File: src/my_robot_description/urdf/urdf/parameter.xacro (robot description, xacro)
@@ -1,4 +1,5 @@
 <?xml version="1.0"?>
 <robot xmlns:xacro="http://www.ros.org/wiki/xacro">
+    <!-- Color properties -->
     <xacro:property name="name_color_base" value="blue"/>
     <xacro:property name="rgba_base" value="0 0 1 1"/>
@@ -15,3 +16,17 @@
     <xacro:property name="name_color_lidar" value="Pinkish_red"/>
     <xacro:property name="rgba_lidar" value="1 0.4 0.4 1"/>
+    <!-- mass properties -->
+    <xacro:property name="mass_base" value="0.5"/>
+    <xacro:property name="mass_base_cap" value="0.2"/>
+    <xacro:property name="mass_body_cover_1" value="0.05"/>
+    <xacro:property name="mass_body_cover_2" value="0.04"/>
+    <xacro:property name="mass_body_cover_3" value="0.08"/>
+    <xacro:property name="mass_body_cover_4" value="0.08"/>
+    <xacro:property name="mass_body" value="1.5"/>
+    <xacro:property name="mass_12V_DC_motor" value="0.1"/>
+    <xacro:property name="mass_altavoz_3" value="0.005"/>
+    <xacro:property name="mass_elp_1080p_modulo" value="0.005"/>
+    <xacro:property name="mass_matriz_de_microfono_resaker_12v" value="0.005"/>
+    <xacro:property name="mass_pantalla_10" value="0.01"/>
+    <xacro:property name="mass_lidar_rplidar" value="0.2"/>
 </robot>

File: src/my_robot_description/urdf/urdf/robot.xacro (robot description, xacro)
@@ -27,4 +27,5 @@
         name_folder="robot_body"
         stl_path="$(arg stl_path)"
+        mass="${mass_base}"
     />
     <!-- Engine -->
@@ -38,4 +39,5 @@
         name_folder="electronics"
         stl_path="$(arg stl_path)"
+        mass="${mass_12V_DC_motor}"
     />
     <xacro:create_link
@@ -48,4 +50,5 @@
         name_folder="electronics"
         stl_path="$(arg stl_path)"
+        mass="${mass_12V_DC_motor}"
     />
     <xacro:create_link
@@ -58,4 +61,5 @@
         name_folder="electronics"
         stl_path="$(arg stl_path)"
+        mass="${mass_12V_DC_motor}"
     />
     <xacro:create_link
@@ -68,4 +72,5 @@
         name_folder="electronics"
         stl_path="$(arg stl_path)"
+        mass="${mass_12V_DC_motor}"
     />
     <!-- Electronics -->
@@ -79,4 +84,5 @@
         name_folder="electronics"
         stl_path="$(arg stl_path)"
+        mass="${mass_pantalla_10}"
     />
     <xacro:create_link
@@ -89,4 +95,5 @@
         name_folder="electronics"
         stl_path="$(arg stl_path)"
+        mass="${mass_altavoz_3}"
     />
     <xacro:create_link
@@ -99,4 +106,5 @@
         name_folder="electronics"
         stl_path="$(arg stl_path)"
+        mass="${mass_altavoz_3}"
     />
     <xacro:create_link
@@ -109,4 +117,5 @@
         name_folder="electronics"
         stl_path="$(arg stl_path)"
+        mass="${mass_elp_1080p_modulo}"
     />
     <xacro:create_link
@@ -119,4 +128,5 @@
         name_folder="electronics"
         stl_path="$(arg stl_path)"
+        mass="${mass_matriz_de_microfono_resaker_12v}"
     />
     <xacro:create_link
@@ -129,4 +139,5 @@
         name_folder="electronics"
         stl_path="$(arg stl_path)"
+        mass="${mass_matriz_de_microfono_resaker_12v}"
     />
     <xacro:create_link
@@ -139,4 +150,5 @@
         name_folder="electronics"
         stl_path="$(arg stl_path)"
+        mass="${mass_lidar_rplidar}"
     />
     <!-- Wheels -->
@@ -191,4 +203,5 @@
         name_folder="robot_body"
         stl_path="$(arg stl_path)"
+        mass="${mass_body}"
     />
     <xacro:create_link
@@ -201,4 +214,5 @@
         name_folder="robot_body"
         stl_path="$(arg stl_path)"
+        mass="${mass_base_cap}"
     />
     <xacro:create_link
@@ -211,4 +225,5 @@
         name_folder="robot_body"
         stl_path="$(arg stl_path)"
+        mass="${mass_body_cover_4}"
     />
     <xacro:create_link
@@ -221,4 +236,5 @@
         name_folder="robot_body"
         stl_path="$(arg stl_path)"
+        mass="${mass_body_cover_3}"
     />
     <xacro:create_link
@@ -231,4 +247,5 @@
         name_folder="robot_body"
         stl_path="$(arg stl_path)"
+        mass="${mass_body_cover_2}"
     />
     <xacro:create_link
@@ -241,4 +258,5 @@
         name_folder="robot_body"
         stl_path="$(arg stl_path)"
+        mass="${mass_body_cover_1}"
     />
     <!-- Joints fijos -->
