Commit message: Refactor macro.xacro and robot.xacro to remove unused stl_path argument; update mesh filenames for improved file management and consistency

File: src/my_robot_description/urdf/urdf/macro.xacro (robot description, xacro)
@@ -1,10 +1,10 @@
 <?xml version="1.0" ?>
 <robot name="my_robot" xmlns:xacro="http://www.ros.org/wiki/xacro">
-    <xacro:macro name="create_link" params="name name_link name_folder name_color rgba xyz rpy stl_path mass">
+    <xacro:macro name="create_link" params="name name_link name_folder name_color rgba xyz rpy mass">
         <link name="${name_link}">
             <visual>
                 <origin xyz="${xyz}" rpy="${rpy}"/>
                 <geometry>
-                    <mesh filename="${stl_path}/${name_folder}/${name}.stl" scale="0.001 0.001 0.001"/>
+                    <mesh filename="package://my_robot_description/urdf/stl/${name_folder}/${name}.stl" scale="0.001 0.001 0.001"/>
                 </geometry>
                 <material name="${name_color}">
@@ -15,5 +15,5 @@
                 <origin xyz="${xyz}" rpy="${rpy}"/>
                 <geometry>
-                    <mesh filename="${stl_path}/${name_folder}/${name}.stl" scale="0.001 0.001 0.001"/>
+                    <mesh filename="package://my_robot_description/urdf/stl/${name_folder}/${name}.stl" scale="0.001 0.001 0.001"/>
                 </geometry>
             </collision>
@@ -25,10 +25,10 @@
         </link>
     </xacro:macro>
-    <xacro:macro name="create_link_wheel" params="name name_link name_folder name_color rgba xyz_collition rpy stl_path">
+    <xacro:macro name="create_link_wheel" params="name name_link name_folder name_color rgba xyz_collition">
         <link name="${name_link}">
             <visual>
                 <origin xyz="0 0 0" rpy="0 0 0"/>
                 <geometry>
-                    <mesh filename="${stl_path}/${name_folder}/${name}.stl" scale="0.001 0.001 0.001"/>
+                    <mesh filename="package://my_robot_description/urdf/stl/${name_folder}/${name}.stl" scale="0.001 0.001 0.001"/>
                 </geometry>
                 <material name="${name_color}">
@@ -37,16 +37,23 @@
             </visual>
             <collision>
-                <origin xyz="${xyz_collition}" rpy="${rpy}"/>
+                <origin xyz="${xyz_collition}" rpy="1.5708 0 0"/>
                 <geometry>
-                    <cylinder length="0.045674" radius="0.028885"/>
+                    <cylinder length="0.045674"
+                            radius="0.028885"/>
                 </geometry>
             </collision>
             <inertial>
-                <mass value="0.045267"/>
+                <mass value="0.3"/>
                 <origin xyz="0 0 0" rpy="0 0 0"/>
-                <inertia ixx="0.001" ixy="0.0" ixz="0.0" iyy="0.001" iyz="0.0" izz="0.001"/>
+                <inertia
+                    ixx="0.0002"
+                    ixy="0.0"
+                    ixz="0.0"
+                    iyy="0.0002"
+                    iyz="0.0"
+                    izz="0.0001"/>
             </inertial>
         </link>
-    </xacro:macro>
+</xacro:macro>
     <xacro:macro name="create_joint_fixed" params="name parent child xyz rpy">
         <joint name="${name}" type="fixed">

File: src/my_robot_description/urdf/urdf/robot.xacro (robot description, xacro)
@@ -4,7 +4,4 @@
     <!-- ARGUMENTOS -->
     <!-- ===================================================== -->
-    <xacro:arg
-        name="stl_path"
-        default="$(find my_robot_description)/urdf/stl"/>
     <xacro:arg
         name="controllers_file"
@@ -26,5 +23,4 @@
         rpy="1.5708 0 0"
         name_folder="robot_body"
-        stl_path="$(arg stl_path)"
         mass="${mass_base}"
     />
@@ -38,5 +34,4 @@
         rpy="0 0 3.14159"
         name_folder="electronics"
-        stl_path="$(arg stl_path)"
         mass="${mass_12V_DC_motor}"
     />
@@ -49,5 +44,4 @@
         rpy="0 0 3.14159"
         name_folder="electronics"
-        stl_path="$(arg stl_path)"
         mass="${mass_12V_DC_motor}"
     />
@@ -60,5 +54,4 @@
         rpy="0 0 0"
         name_folder="electronics"
-        stl_path="$(arg stl_path)"
         mass="${mass_12V_DC_motor}"
     />
@@ -71,5 +64,4 @@
         rpy="0 0 0"
         name_folder="electronics"
-        stl_path="$(arg stl_path)"
         mass="${mass_12V_DC_motor}"
     />
@@ -83,5 +75,4 @@
         rpy="0 1.5708 1.5708"
         name_folder="electronics"
-        stl_path="$(arg stl_path)"
         mass="${mass_pantalla_10}"
     />
@@ -94,5 +85,4 @@
         rpy="0 0 3.14159"
         name_folder="electronics"
-        stl_path="$(arg stl_path)"
         mass="${mass_altavoz_3}"
     />
@@ -105,5 +95,4 @@
         rpy="0 0 0"
         name_folder="electronics"
-        stl_path="$(arg stl_path)"
         mass="${mass_altavoz_3}"
     />
@@ -116,5 +105,4 @@
         rpy="0 0 1.5708"
         name_folder="electronics"
-        stl_path="$(arg stl_path)"
         mass="${mass_elp_1080p_modulo}"
     />
@@ -127,5 +115,4 @@
         rpy="1.5708 0 0"
         name_folder="electronics"
-        stl_path="$(arg stl_path)"
         mass="${mass_matriz_de_microfono_resaker_12v}"
     />
@@ -138,5 +125,4 @@
         rpy="1.5708 0 0"
         name_folder="electronics"
-        stl_path="$(arg stl_path)"
         mass="${mass_matriz_de_microfono_resaker_12v}"
     />
@@ -149,5 +135,4 @@
         rpy="1.5708 0 0"
         name_folder="electronics"
-        stl_path="$(arg stl_path)"
         mass="${mass_lidar_rplidar}"
     />
@@ -158,8 +143,6 @@
         name_color="${name_color_wheel}"
         rgba="${rgba_wheel}"
-        rpy="0 0 0"
         name_folder="robot_body"
         xyz_collition="0 0.065 0"
-        stl_path="$(arg stl_path)"
     />
     <xacro:create_link_wheel
@@ -168,8 +151,6 @@
         name_color="${name_color_wheel}"
         rgba="${rgba_wheel}"
-        rpy="0 0 3.14159"
         name_folder="robot_body"
         xyz_collition="0 0.07 0"
-        stl_path="$(arg stl_path)"
     />
     <xacro:create_link_wheel
@@ -178,8 +159,6 @@
         name_color="${name_color_wheel}"
         rgba="${rgba_wheel}"
-        rpy="0 0 0"
         name_folder="robot_body"
         xyz_collition="0 0.05 0"
-        stl_path="$(arg stl_path)"
     />
     <xacro:create_link_wheel
@@ -188,8 +167,6 @@
         name_color="${name_color_wheel}"
         rgba="${rgba_wheel}"
-        rpy="0 0 3.14159"
         name_folder="robot_body"
         xyz_collition="0 0.05 0"
-        stl_path="$(arg stl_path)"
     />
     <!-- Body covers -->
@@ -202,5 +179,4 @@
         rpy="1.5708 0 -1.5708"
         name_folder="robot_body"
-        stl_path="$(arg stl_path)"
         mass="${mass_body}"
     />
@@ -213,5 +189,4 @@
         rpy="0 3.14159 1.5708"
         name_folder="robot_body"
-        stl_path="$(arg stl_path)"
         mass="${mass_base_cap}"
     />
@@ -224,5 +199,4 @@
         rpy="0 3.14159 -1.5708"
         name_folder="robot_body"
-        stl_path="$(arg stl_path)"
         mass="${mass_body_cover_4}"
     />
@@ -235,5 +209,4 @@
         rpy="-1.5708 -1.5708 0"
         name_folder="robot_body"
-        stl_path="$(arg stl_path)"
         mass="${mass_body_cover_3}"
     />
@@ -246,5 +219,4 @@
         rpy="-1.5708 -1.5708 0"
         name_folder="robot_body"
-        stl_path="$(arg stl_path)"
         mass="${mass_body_cover_2}"
     />
@@ -257,5 +229,4 @@
         rpy="0 0 -1.5708"
         name_folder="robot_body"
-        stl_path="$(arg stl_path)"
         mass="${mass_body_cover_1}"
     />
@@ -383,5 +354,5 @@
     <xacro:create_joint_continuous
     name="base_link_to_right_wheel_2"
-    parent="engine_2_link"
+    parent="base_link"
     child="right_wheel_1_link"
     xyz="-0.240 -0.263 0.023"
@@ -391,5 +362,5 @@
     <xacro:create_joint_continuous
     name="base_link_to_right_wheel_3"
-    parent="engine_3_link"
+    parent="base_link"
     child="right_wheel_2_link"
     xyz="0.240 0.263 0.023"
@@ -399,5 +370,5 @@
     <xacro:create_joint_continuous
     name="base_link_to_left_wheel_1"
-    parent="engine_1_link"
+    parent="base_link"
     child="left_wheel_1_link"
     xyz="0.240 -0.243 0.023"
@@ -407,5 +378,5 @@
     <xacro:create_joint_continuous
     name="base_link_to_left_wheel_4"
-    parent="engine_4_link"
+    parent="base_link"
     child="left_wheel_2_link"
     xyz="-0.240 0.243 0.023"
