Commit message: Add event handlers for joint state broadcaster and diff drive controller in gazebo launch file; update robot.xacro with base footprint link and joint definition

File: kairo_sim/src/my_robot_description/urdf/urdf/robot.xacro (robot description, xacro)
@@ -14,4 +14,6 @@
     <xacro:include filename="./ros2_control.xacro"/>
     <xacro:include filename="./gazebo.xacro"/>
+    <!-- Robot links -->
+    <link name="base_footprint"/>
     <!-- link Base -->
     <xacro:create_link
@@ -232,4 +234,9 @@
     />
     <!-- Joints fijos -->
+    <joint name="base_footprint_to_base_link" type="fixed">
+        <parent link="base_footprint"/>
+        <child link="base_link"/>
+        <origin xyz="0 0 0.023" rpy="0 0 0"/>
+    </joint>
     <xacro:create_joint_fixed
     name="base_link_to_base_cap"

Commit message: Fix joint origin position for base_footprint to base_link in robot.xacro

File: kairo_sim/src/my_robot_description/urdf/urdf/robot.xacro (robot description, xacro)
@@ -237,5 +237,5 @@
         <parent link="base_footprint"/>
         <child link="base_link"/>
-        <origin xyz="0 0 0.023" rpy="0 0 0"/>
+        <origin xyz="0 0 0" rpy="0 0 0"/>
     </joint>
     <xacro:create_joint_fixed
