Commit message: Update controllers and launch files; add LIDAR and IMU sensors to robot description

File: kairo_sim/src/my_robot_description/urdf/urdf/gazebo.xacro (robot description, xacro)
@@ -61,3 +61,39 @@
         <material>Gazebo/Grey</material>
     </gazebo>
+    <!-- ===================================================== -->
+    <!-- LIDAR -->
+    <!-- ===================================================== -->
+    <gazebo reference="sensor_lidar_link">
+        <sensor name="lidar_sensor" type="lidar">
+            <always_on>true</always_on>
+            <visualize>true</visualize>
+            <update_rate>10</update_rate>
+            <topic>/scan</topic>
+            <lidar>
+                <scan>
+                    <horizontal>
+                        <samples>360</samples>
+                        <resolution>1</resolution>
+                        <min_angle>-3.14159</min_angle>
+                        <max_angle>3.14159</max_angle>
+                    </horizontal>
+                </scan>
+                <range>
+                    <min>0.10</min>
+                    <max>10.0</max>
+                    <resolution>0.01</resolution>
+                </range>
+            </lidar>
+        </sensor>
+    </gazebo>
+    <!-- ===================================================== -->
+    <!-- IMU -->
+    <!-- ===================================================== -->
+    <gazebo reference="imu_link">
+        <sensor name="imu_sensor" type="imu">
+            <always_on>true</always_on>
+            <update_rate>100</update_rate>
+            <topic>/imu</topic>
+        </sensor>
+    </gazebo>
 </robot>

File: kairo_sim/src/my_robot_description/urdf/urdf/robot.xacro (robot description, xacro)
@@ -129,14 +129,58 @@
         mass="${mass_matriz_de_microfono_resaker_12v}"
     />
-    <xacro:create_link
-        name="sensor_lidar"
-        name_link="sensor_lidar_link"
-        name_color="${name_color_lidar}"
-        rgba="${rgba_lidar}"
-        xyz="-0.18 0 1.24"
-        rpy="1.5708 0 0"
-        name_folder="electronics"
-        mass="${mass_lidar_rplidar}"
-    />
+    <link name="sensor_lidar_link">
+        <visual>
+            <origin xyz="0 0 0" rpy="0 0 0"/>
+            <geometry>
+                <cylinder radius="0.04" length="0.05"/>
+            </geometry>
+            <material name="black">
+                <color rgba="0 0 0 1"/>
+            </material>
+        </visual>
+        <collision>
+            <origin xyz="0 0 0" rpy="0 0 0"/>
+            <geometry>
+                <cylinder radius="0.04" length="0.05"/>
+            </geometry>
+        </collision>
+        <inertial>
+            <mass value="0.1"/>
+            <origin xyz="0 0 0" rpy="0 0 0"/>
+            <inertia
+                ixx="0.001"
+                ixy="0"
+                ixz="0"
+                iyy="0.001"
+                iyz="0"
+                izz="0.001"/>
+        </inertial>
+    </link>
+    <link name="imu_link">
+        <visual>
+            <geometry>
+                <box size="0.03 0.03 0.01"/>
+            </geometry>
+            <material name="blue">
+                <color rgba="0 0 1 1"/>
+            </material>
+        </visual>
+        <collision>
+            <geometry>
+                <box size="0.03 0.03 0.01"/>
+            </geometry>
+        </collision>
+        <inertial>
+            <mass value="0.01"/>
+            <origin xyz="0 0 0" rpy="0 0 0"/>
+            <inertia
+                ixx="0.0001"
+                ixy="0"
+                ixz="0"
+                iyy="0.0001"
+                iyz="0"
+                izz="0.0001"/>
+        </inertial>
+    </link>
     <!-- Wheels -->
     <xacro:create_link_wheel
@@ -391,3 +435,10 @@
     axis="0 -1 0"
     />
+    <xacro:create_joint_fixed
+    name="base_link_to_imu"
+    parent="base_link"
+    child="imu_link"
+    xyz="0 0 0"
+    rpy="0 0 0"
+    />
 </robot>

Commit message: Refactor sensor bridge in gazebo.launch.py; update lidar sensor type to gpu_lidar and add IMU sensor configuration in gazebo.xacro; adjust robot origin in robot.xacro; integrate sensors plugin in ros2_control.xacro and world_restauran.sdf

File: kairo_sim/src/my_robot_description/urdf/urdf/gazebo.xacro (robot description, xacro)
@@ -65,9 +65,10 @@
     <!-- ===================================================== -->
     <gazebo reference="sensor_lidar_link">
-        <sensor name="lidar_sensor" type="lidar">
+        <sensor name="lidar_sensor" type="gpu_lidar">
             <always_on>true</always_on>
             <visualize>true</visualize>
             <update_rate>10</update_rate>
             <topic>/scan</topic>
+            <gz_frame_id>sensor_lidar_link</gz_frame_id>
             <lidar>
                 <scan>
@@ -94,5 +95,49 @@
             <always_on>true</always_on>
             <update_rate>100</update_rate>
+            <visualize>true</visualize>
             <topic>/imu</topic>
+            <gz_frame_id>imu_link</gz_frame_id>
+            <imu>
+                <angular_velocity>
+                    <x>
+                        <noise type="gaussian">
+                            <mean>0.0</mean>
+                            <stddev>0.0002</stddev>
+                        </noise>
+                    </x>
+                    <y>
+                        <noise type="gaussian">
+                            <mean>0.0</mean>
+                            <stddev>0.0002</stddev>
+                        </noise>
+                    </y>
+                    <z>
+                        <noise type="gaussian">
+                            <mean>0.0</mean>
+                            <stddev>0.0002</stddev>
+                        </noise>
+                    </z>
+                </angular_velocity>
+                <linear_acceleration>
+                    <x>
+                        <noise type="gaussian">
+                            <mean>0.0</mean>
+                            <stddev>0.017</stddev>
+                        </noise>
+                    </x>
+                    <y>
+                        <noise type="gaussian">
+                            <mean>0.0</mean>
+                            <stddev>0.017</stddev>
+                        </noise>
+                    </y>
+                    <z>
+                        <noise type="gaussian">
+                            <mean>0.0</mean>
+                            <stddev>0.017</stddev>
+                        </noise>
+                    </z>
+                </linear_acceleration>
+            </imu>
         </sensor>
     </gazebo>

File: kairo_sim/src/my_robot_description/urdf/urdf/robot.xacro (robot description, xacro)
@@ -173,5 +173,5 @@
         <inertial>
             <mass value="0.01"/>
-            <origin xyz="0 0 0" rpy="0 0 0"/>
+            <origin xyz="-0.18 0 1.24" rpy="1.5708 0 0"/>
             <inertia
                 ixx="0.0001"

File: kairo_sim/src/my_robot_description/urdf/urdf/ros2_control.xacro (robot description, xacro)
@@ -4,4 +4,8 @@
         <hardware>
             <plugin>gz_ros2_control/GazeboSimSystem</plugin>
+            <plugin
+                filename="gz-sim-sensors-system"
+                name="gz::sim::systems::Sensors"
+            />
         </hardware>
         <!-- ============================================== -->

Commit message: Enhance robot description by updating lidar and imu sensor configurations; adjust sensor properties and add IMU plugin to world SDF

File: kairo_sim/src/my_robot_description/urdf/urdf/gazebo.xacro (robot description, xacro)
@@ -66,7 +66,8 @@
     <gazebo reference="sensor_lidar_link">
         <sensor name="lidar_sensor" type="gpu_lidar">
-            <always_on>true</always_on>
-            <visualize>true</visualize>
-            <update_rate>10</update_rate>
+            <pose realative_to="sensor_lidar_link">0 0 0 0 0 0</pose>
+            <always_on>1</always_on>
+            <visualize>1</visualize>
+            <update_rate>2</update_rate>
             <topic>/scan</topic>
             <gz_frame_id>sensor_lidar_link</gz_frame_id>
@@ -74,5 +75,5 @@
                 <scan>
                     <horizontal>
-                        <samples>360</samples>
+                        <samples>720</samples>
                         <resolution>1</resolution>
                         <min_angle>-3.14159</min_angle>
@@ -83,6 +84,11 @@
                     <min>0.10</min>
                     <max>10.0</max>
-                    <resolution>0.01</resolution>
+                    <resolution>0.005</resolution>
                 </range>
+                <noise>
+                    <type>gaussian</type>
+                    <mean>0.0</mean>
+                    <stddev>0.001</stddev>
+                </noise>
             </lidar>
         </sensor>
@@ -93,9 +99,8 @@
     <gazebo reference="imu_link">
         <sensor name="imu_sensor" type="imu">
-            <always_on>true</always_on>
+            <always_on>1</always_on>
             <update_rate>100</update_rate>
             <visualize>true</visualize>
             <topic>/imu</topic>
-            <gz_frame_id>imu_link</gz_frame_id>
             <imu>
                 <angular_velocity>

File: kairo_sim/src/my_robot_description/urdf/urdf/robot.xacro (robot description, xacro)
@@ -131,7 +131,6 @@
     <link name="sensor_lidar_link">
         <visual>
-            <origin xyz="0 0 0" rpy="0 0 0"/>
             <geometry>
-                <cylinder radius="0.04" length="0.05"/>
+                <cylinder radius="0.035" length="0.05"/>
             </geometry>
             <material name="black">
@@ -140,7 +139,6 @@
         </visual>
         <collision>
-            <origin xyz="0 0 0" rpy="0 0 0"/>
             <geometry>
-                <cylinder radius="0.04" length="0.05"/>
+                <cylinder radius="0.035" length="0.05"/>
             </geometry>
         </collision>
@@ -160,25 +158,25 @@
         <visual>
             <geometry>
-                <box size="0.03 0.03 0.01"/>
+                <box size="0.03 0.03 0.02"/>
             </geometry>
-            <material name="blue">
-                <color rgba="0 0 1 1"/>
+            <material name="gray">
+                <color rgba="0.5 0.5 0.5 1"/>
             </material>
         </visual>
         <collision>
             <geometry>
-                <box size="0.03 0.03 0.01"/>
+                <box size="0.03 0.03 0.02"/>
             </geometry>
         </collision>
         <inertial>
-            <mass value="0.01"/>
-            <origin xyz="-0.18 0 1.24" rpy="1.5708 0 0"/>
+            <mass value="0.05"/>
+            <origin xyz="0 0 0" rpy="0 0 0"/>
             <inertia
-                ixx="0.0001"
+                ixx="1e-5"
                 ixy="0"
                 ixz="0"
-                iyy="0.0001"
+                iyy="1e-5"
                 iyz="0"
-                izz="0.0001"/>
+                izz="1e-5"/>
         </inertial>
     </link>
@@ -399,5 +397,12 @@
     parent="base_link"
     child="sensor_lidar_link"
-    xyz="0 0 0"
+    xyz="-0.18 0 1.32"
+    rpy="0 0 0"
+    />
+    <xacro:create_joint_fixed
+    name="base_link_to_imu"
+    parent="base_link"
+    child="imu_link"
+    xyz="0.0 0 1.25"
     rpy="0 0 0"
     />
@@ -435,10 +440,3 @@
     axis="0 -1 0"
     />
-    <xacro:create_joint_fixed
-    name="base_link_to_imu"
-    parent="base_link"
-    child="imu_link"
-    xyz="0 0 0"
-    rpy="0 0 0"
-    />
 </robot>
